File: Amstrad_PPC_Internal_Expansion/Kicad/Amstrad_PPC_Internal_CF_Lite.kicad_sch (KiCad schematic)
At the start: 36 parts, among them J1 Amstrad_PPC_ISA_Connector_B, J2 Amstrad_PPC_ISA_Connector_A, J3 CONN_CF_CARD, J4 Conn_01x02, SW1 Switch_DIP_4_Positions, SW2 Switch_DIP_8_Positions, U1 74HCT244, U2 74HCT244, U3 74HCT688, U4 74LS32, U5 74HCT04, U6 74HCT688, U7 28C256

Commit message: Starting again ... initial schematic cleanup
Schematic is now cleaned up, no errors
Next will be PCB layout
Parts:
- removed D1: LED, Connector_PinHeader_2.54mm:PinHeader_1x02_P2.54mm_Vertical, symbol Device:LED
- removed HOLE1, HOLE2, HOLE3, HOLE4: HOLE, My_Components:Hole_3mm, symbol my_components:HOLE
- removed J3: CONN_CF_CARD, My_Components:Conn_CF_N7E50-Q516XX-40, symbol my_components:CONN_CF_CARD
- removed RR1: 10KΩ, Resistor_THT:R_Array_SIP10, symbol my_components:RR9
- removed SW1: Switch_DIP_4_Positions, My_Components:Switch_DIP_4_Positions, symbol my_components:Switch_DIP_4_Positions
- removed SW2: Switch_DIP_8_Positions, My_Components:Switch_DIP_8_Positions, symbol my_components:Switch_DIP_8_Positions
- removed U7: 28C256, Package_DIP:DIP-28_W15.24mm, symbol my_components:28C256
- added H1, H2, H3, H4: MountingHole_Pad, MountingHole:MountingHole_6.4mm_M6_DIN965_Pad, symbol Mechanical:MountingHole_Pad
- added J3: LED, Connector_PinHeader_2.54mm:PinHeader_1x02_P2.54mm_Vertical, symbol Connector_Generic:Conn_01x02
- added J5: N7E50-Q516RB-50-WF, Amstrad_PPC:N7E50Q516RB50WF, symbol Amstrad_PPC:N7E50-Q516RB-50-WF
- added RN2: 10KΩ, Resistor_THT:R_Array_SIP9, symbol Device:R_Network08
- added SW2: SW_DIP_x04, Button_Switch_THT:SW_DIP_SPSTx04_Slide_9.78x12.34mm_W7.62mm_P2.54mm, symbol Switch:SW_DIP_x04
- added SW3: SW_DIP_x08, Button_Switch_THT:SW_DIP_SPSTx08_Slide_9.78x22.5mm_W7.62mm_P2.54mm, symbol Switch:SW_DIP_x08
- added U8: 28C256, Package_DIP:DIP-28_W15.24mm_Socket, symbol Memory_EEPROM:28C256
- C1, C2, C3, C4, C5, C6, C7: footprint Capacitor_THT:C_Disc_D4.7mm_W2.5mm_P5.00mm -> Capacitor_THT:C_Disc_D3.4mm_W2.1mm_P2.50mm
- C8: footprint Capacitor_THT:C_Radial_D4.0mm_H5.0mm_P1.50mm -> Capacitor_THT:CP_Radial_D5.0mm_P2.50mm
- J1: footprint Connector_Dsub:DSUB-37_Female_EdgeMount_P2.77mm -> Connector_Dsub:DSUB-37_Socket_EdgeMount_P2.77mm; symbol Connector:Amstrad_PPC_ISA_Connector_B -> Amstrad_PPC:Amstrad_PPC_ISA_Connector_B
- J2: footprint Connector_Dsub:DSUB-25_Female_EdgeMount_P2.77mm -> Connector_Dsub:DSUB-25_Socket_EdgeMount_P2.77mm; symbol Connector:Amstrad_PPC_ISA_Connector_A -> Amstrad_PPC:Amstrad_PPC_ISA_Connector_A
- J4: value Conn_01x02 -> LED
- U4: value 74LS32 -> 74HCT32
Connections:
- net B_A08 is gone; now on net A_{08}: U3.8 (P3)
- net B_RESET: now also U5.3
- net CF_DMARQ: now also R5.1, J5.43 (DMREQ); no longer R5.2
- net CF_IORDY: now also J5.42 (IORDY)
- net GND: now also R5.2, H1.1, H2.1, H3.1, H4.1, J5.1 (GND), J5.10 (A9), J5.11 (A8), J5.12 (A7), J5.14 (A6), J5.15 (A5), J5.16 (A4), J5.17 (A3), J5.39 (~{CSEL}), J5.50 (GND), J5.8 (A10), J5.9 (~{ATA}), J5.MH1, J5.MH2, J5.MP1, J5.MP2, SW2.6, SW2.7, SW2.8, SW3.1, SW3.3, SW3.4, SW3.5, SW3.6, SW3.7, U8.1 (A14), U8.14 (GND), U8.26 (A13); no longer R5.1
- net VCC: now also J5.13 (V_{CC}), J5.36 (~{WE}), J5.38 (V_{CC}), J5.44 (~{DMACK}), RN2.1 (common), U8.28 (VCC)
- net ~{B_IOR}: now also J5.34 (~{IORD})
- net ~{B_IOW}: now also J5.35 (~{IOWR})
- net ~{B_MEMR}: now also U8.22 (~{OE})
- net ~{B_MEMW}: now also SW3.2
- net ~{CF_CS0}: now also J5.7 (~{CS0})
- net ~{CF_CS1}: now also J5.32 (~{CS1})
- net ~{CF_DASP}: now also J5.45 (~{DASP})
- net ~{ROMW}: now also RN2.3 (R2), SW3.15, U8.27 (~{WE})
- net ~{ROM_CS}: now also U8.20 (~{CS})
- net at U6.1 (G): now also RN2.2 (R1), SW3.16
- net at U6.7 (R2): now also RN2.4 (R3), SW3.14
- net at U6.9 (R3): now also RN2.5 (R4), SW3.13
- net at U6.12 (R4): now also RN2.6 (R5), SW3.12
- net at U6.14 (R5): now also RN2.7 (R6), SW3.11
- net at U6.16 (R6): now also RN2.8 (R7), SW3.10
- net at R7.2: now also J3.1 (Pin_1)
- net at R3.2, U3.7 (R2): now also SW2.1
- net at U5.8: now also J3.2 (Pin_2)
- net at R2.2, U3.5 (R1): now also SW2.2
- net at R1.2, U3.3 (R0): now also SW2.3
- net A00 renamed A_{00}
- net A_{00}: now also U1.2 (1A0); no longer U1.11 (2A3)
- net A01 renamed A_{01}
- net A_{01}: now also U1.4 (1A1); no longer U1.8 (1A3)
- net A02 renamed A_{02}
- net A_{02}: now also U1.6 (1A2); no longer U1.13 (2A2)
- net A03 renamed A_{03}
- net A_{03}: now also U1.8 (1A3); no longer U1.6 (1A2)
- net A04 renamed A_{04}
- net A_{04}: now also U1.17 (2A0); no longer U1.15 (2A1)
- net A05 renamed A_{05}
- net A_{05}: now also U1.15 (2A1); no longer U1.4 (1A1)
- net A06 renamed A_{06}
- net A_{06}: now also U1.13 (2A2); no longer U1.17 (2A0)
- net A07 renamed A_{07}
- net A_{07}: now also U1.11 (2A3); no longer U1.2 (1A0)
- net A08 renamed A_{08}
- net A_{08}: now also U8.25 (A8)
- net A09 renamed A_{09}
- net A_{09}: now also U8.24 (A9)
- net A10 renamed A_{10}
- net A_{10}: now also U8.21 (A10)
- net A11 renamed A_{11}
- net A_{11}: now also U8.23 (A11)
- net A12 renamed A_{12}
- net A_{12}: now also U8.2 (A12)
- net A13 renamed A_{13}
- net A14 renamed A_{14}
- net A15 renamed A_{15}
- net A16 renamed A_{16}
- net A17 renamed A_{17}
- net A18 renamed A_{18}
- net A19 renamed A_{19}
- net B_A00 renamed B_A_{07}
- net B_A_{07}: now also U3.6 (P2), U8.3 (A7)
- net B_A01 renamed B_A_{03}
- net B_A_{03}: now also U8.7 (A3)
- net B_A02 renamed B_A_{06}
- net B_A_{06}: now also U3.4 (P1), U8.4 (A6)
- net B_A03 renamed B_A_{02}
- net B_A_{02}: now also J5.18 (A2), U8.8 (A2)
- net B_A04 renamed B_A_{04}
- net B_A_{04}: now also U1.3 (2Y0), U8.6 (A4); no longer U1.5 (2Y1)
- net B_A05 renamed B_A_{01}
- net B_A_{01}: now also J5.19 (A1), U8.9 (A1); no longer U3.2 (P0)
- removed net B_A06: U1.3 (2Y0), U3.4 (P1)
- net B_A07 renamed B_A_{00}
- net B_A_{00}: now also J5.20 (A0), U8.10 (A0); no longer U3.6 (P2)
- net D0 renamed D_{0}
- net D_{0}: now also J5.21 (D0), U8.11 (D0)
- net D1 renamed D_{1}
- net D_{1}: now also J5.22 (D1), U8.12 (D1)
- net D2 renamed D_{2}
- net D_{2}: now also J5.23 (D2), U8.13 (D2)
- net D3 renamed D_{3}
- net D_{3}: now also J5.2 (D3), U8.15 (D3)
- net D4 renamed D_{4}
- net D_{4}: now also J5.3 (D4), U8.16 (D4)
- net D5 renamed D_{5}
- net D_{5}: now also J5.4 (D5), U8.17 (D5)
- net D6 renamed D_{6}
- net D_{6}: now also J5.5 (D6), U8.18 (D6)
- net D7 renamed D_{7}
- net D_{7}: now also J5.6 (D7), U8.19 (D7)
- net ~{CF_RESET} renamed ~{B_RESET}
- net ~{B_RESET}: now also J5.41 (~{RESET})
- new net B_A_{05}: U1.5 (2Y1), U3.2 (P0), U8.5 (A5)
- no-connect marks 51 -> 50
Other:
- note removed: "BIOS Extension ROM"
- note removed: "Bypass Capacitors"
- note removed: "Data signal pullup"
- note removed: "MODEM Board Mounting Holes"
- moved on the sheet: J2, J4, R4, R5, R6, R7, R8, U5B, U5C, U5D, U5E, U5F
