File: Amstrad_PPC_Internal_Expansion/Kicad/Amstrad_PPC_Internal_CF_Lite.kicad_sch (KiCad schematic)
At the start: 36 parts, among them J1 Amstrad_PPC_ISA_Connector_B, J2 Amstrad_PPC_ISA_Connector_A, J3 LED, J4 LED, J5 N7E50-Q516RB-50-WF, SW2 SW_DIP_x04, SW3 SW_DIP_x08, U1 74HCT244, U2 74HCT244, U3 74HCT688, U4 74HCT32, U5 74HCT04, U6 74HCT688, U8 28C256

Commit message: Update Amstrad_PPC_Internal_CF_Lite.kicad_sch
Parts:
- added H5, H6, H7: MountingHole_Pad, MountingHole:MountingHole_3.2mm_M3_DIN965_Pad, symbol Mechanical:MountingHole_Pad
- H3, H4: footprint MountingHole:MountingHole_6.4mm_M6_DIN965_Pad -> MountingHole:MountingHole_3.2mm_M3_DIN965_Pad
Connections:
- net GND: now also H5.1, H6.1, H7.1
Other:
- note removed: "Compact Flash Interface"
- note removed: "Here Be The ISA Expansion Bus"
- note removed: "I/O Port Chip Select Logic"
- note removed: "Signal buffering"
- note removed: "Spares"
- moved on the sheet: C1, C2, C3, C4, C5, C6, C7, C8, H1, H2, H3, H4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
